File: Accelerometer.kicad_sch (KiCad schematic)
At the start: 3 parts, among them U10 LIS3DSHTR

Commit message: finalize
Parts:
- C20: value 10uF -> 10u; footprint Capacitor_SMD:C_0805_2012Metric_Pad1.18x1.45mm_HandSolder -> Capacitor_SMD:C_0805_2012Metric
- C21: value 100nF -> 100n; footprint Capacitor_SMD:C_0805_2012Metric_Pad1.18x1.45mm_HandSolder -> Capacitor_SMD:C_0805_2012Metric
Changed lines of the file:
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@@
 		)
 		(instances
-			(project "meshtastic-v0"
+			(project "meshthingy"
 				(path "/e4d6fcd6-7415-4955-88fd-f0e430797514/5dd6f357-5254-45d8-811a-b64551c52eaf"
 					(reference "#PWR054")
@@
 		)
 		(instances
-			(project "meshtastic-v0"
+			(project "meshthingy"
 				(path "/e4d6fcd6-7415-4955-88fd-f0e430797514/5dd6f357-5254-45d8-811a-b64551c52eaf"
 					(reference "#PWR053")
@@
 		)
 		(instances
-			(project "meshtastic-v0"
+			(project "meshthingy"
 				(path "/e4d6fcd6-7415-4955-88fd-f0e430797514/5dd6f357-5254-45d8-811a-b64551c52eaf"
 					(reference "#PWR052")
@@
 			)
 		)
-		(property "Value" "10uF"
+		(property "Value" "10u"
 			(at 58.42 76.1999 0)
 			(show_name no)
@@
 			)
 		)
-		(property "Footprint" "Capacitor_SMD:C_0805_2012Metric_Pad1.18x1.45mm_HandSolder"
+		(property "Footprint" "Capacitor_SMD:C_0805_2012Metric"
 			(at 55.5752 78.74 0)
 			(hide yes)
@@
 		)
 		(instances
-			(project "meshtastic-v0"
+			(project "meshthingy"
 				(path "/e4d6fcd6-7415-4955-88fd-f0e430797514/5dd6f357-5254-45d8-811a-b64551c52eaf"
 					(reference "C20")
@@
 		)
 		(instances
-			(project "meshtastic-v0"
+			(project "meshthingy"
 				(path "/e4d6fcd6-7415-4955-88fd-f0e430797514/5dd6f357-5254-45d8-811a-b64551c52eaf"
 					(reference "U10")
@@
 		)
 		(instances
-			(project "meshtastic-v0"
+			(project "meshthingy"
 				(path "/e4d6fcd6-7415-4955-88fd-f0e430797514/5dd6f357-5254-45d8-811a-b64551c52eaf"
 					(reference "#PWR055")
@@
 			)
 		)
-		(property "Value" "100nF"
+		(property "Value" "100n"
 			(at 71.12 76.1999 0)
 			(show_name no)
@@
 			)
 		)
-		(property "Footprint" "Capacitor_SMD:C_0805_2012Metric_Pad1.18x1.45mm_HandSolder"
+		(property "Footprint" "Capacitor_SMD:C_0805_2012Metric"
 			(at 68.2752 78.74 0)
 			(hide yes)
@@
 		)
 		(instances
-			(project "meshtastic-v0"
+			(project "meshthingy"
 				(path "/e4d6fcd6-7415-4955-88fd-f0e430797514/5dd6f357-5254-45d8-811a-b64551c52eaf"
 					(reference "C21")
