File: Air Sensors.kicad_sch (KiCad schematic)
At the start: 3 parts, among them U9 BME280

Commit message: finalize
Parts:
- C23, C24: value 100nF -> 100n; footprint Capacitor_SMD:C_0805_2012Metric_Pad1.18x1.45mm_HandSolder -> Capacitor_SMD:C_0805_2012Metric
Changed lines of the file:
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@@
 		)
 		(instances
-			(project "meshtastic-v0"
+			(project "meshthingy"
 				(path "/e4d6fcd6-7415-4955-88fd-f0e430797514/7d370f93-0a3a-4229-8480-c7d167e20db4"
 					(reference "#PWR057")
@@
 		)
 		(instances
-			(project "meshtastic-v0"
+			(project "meshthingy"
 				(path "/e4d6fcd6-7415-4955-88fd-f0e430797514/7d370f93-0a3a-4229-8480-c7d167e20db4"
 					(reference "U9")
@@
 		)
 		(instances
-			(project "meshtastic-v0"
+			(project "meshthingy"
 				(path "/e4d6fcd6-7415-4955-88fd-f0e430797514/7d370f93-0a3a-4229-8480-c7d167e20db4"
 					(reference "#PWR059")
@@
 		)
 		(instances
-			(project "meshtastic-v0"
+			(project "meshthingy"
 				(path "/e4d6fcd6-7415-4955-88fd-f0e430797514/7d370f93-0a3a-4229-8480-c7d167e20db4"
 					(reference "#PWR062")
@@
 			)
 		)
-		(property "Value" "100nF"
+		(property "Value" "100n"
 			(at 69.85 69.8499 0)
 			(show_name no)
@@
 			)
 		)
-		(property "Footprint" "Capacitor_SMD:C_0805_2012Metric_Pad1.18x1.45mm_HandSolder"
+		(property "Footprint" "Capacitor_SMD:C_0805_2012Metric"
 			(at 67.0052 72.39 0)
 			(hide yes)
@@
 		)
 		(instances
-			(project "meshtastic-v0"
+			(project "meshthingy"
 				(path "/e4d6fcd6-7415-4955-88fd-f0e430797514/7d370f93-0a3a-4229-8480-c7d167e20db4"
 					(reference "C23")
@@
 		)
 		(instances
-			(project "meshtastic-v0"
+			(project "meshthingy"
 				(path "/e4d6fcd6-7415-4955-88fd-f0e430797514/7d370f93-0a3a-4229-8480-c7d167e20db4"
 					(reference "#PWR060")
@@
 		)
 		(instances
-			(project "meshtastic-v0"
+			(project "meshthingy"
 				(path "/e4d6fcd6-7415-4955-88fd-f0e430797514/7d370f93-0a3a-4229-8480-c7d167e20db4"
 					(reference "#PWR061")
@@
 			)
 		)
-		(property "Value" "100nF"
+		(property "Value" "100n"
 			(at 82.55 69.8499 0)
 			(show_name no)
@@
 			)
 		)
-		(property "Footprint" "Capacitor_SMD:C_0805_2012Metric_Pad1.18x1.45mm_HandSolder"
+		(property "Footprint" "Capacitor_SMD:C_0805_2012Metric"
 			(at 79.7052 72.39 0)
 			(hide yes)
@@
 		)
 		(instances
-			(project "meshtastic-v0"
+			(project "meshthingy"
 				(path "/e4d6fcd6-7415-4955-88fd-f0e430797514/7d370f93-0a3a-4229-8480-c7d167e20db4"
 					(reference "C24")
