File: Connectors.kicad_sch (KiCad schematic)
At the start: 4 parts, among them J1 USB_C_Receptacle_USB2.0_16P, J2 Conn_01x02_Pin

Commit message: finalize
Parts:
- J1: value USB_C_Receptacle_USB2.0_16P -> USB_C_16P
- J2: value Conn_01x02_Pin -> BATT_Con
Changed lines of the file:
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@@
 			)
 		)
-		(property "Value" "Conn_01x02_Pin"
+		(property "Value" "BATT_Con"
 			(at 39.37 77.978 0)
 			(show_name no)
@@
 		)
 		(instances
-			(project "meshtastic-v0"
+			(project "meshthingy"
 				(path "/e4d6fcd6-7415-4955-88fd-f0e430797514/2c15135a-b809-49e8-b858-375c97ce8d4a"
 					(reference "J2")
@@
 		)
 		(instances
-			(project "meshtastic-v0"
+			(project "meshthingy"
 				(path "/e4d6fcd6-7415-4955-88fd-f0e430797514/2c15135a-b809-49e8-b858-375c97ce8d4a"
 					(reference "#PWR032")
@@
 		)
 		(instances
-			(project "meshtastic-v0"
+			(project "meshthingy"
 				(path "/e4d6fcd6-7415-4955-88fd-f0e430797514/2c15135a-b809-49e8-b858-375c97ce8d4a"
 					(reference "R1")
@@
 		)
 		(instances
-			(project "meshtastic-v0"
+			(project "meshthingy"
 				(path "/e4d6fcd6-7415-4955-88fd-f0e430797514/2c15135a-b809-49e8-b858-375c97ce8d4a"
 					(reference "#PWR010")
@@
 		)
 		(instances
-			(project "meshtastic-v0"
+			(project "meshthingy"
 				(path "/e4d6fcd6-7415-4955-88fd-f0e430797514/2c15135a-b809-49e8-b858-375c97ce8d4a"
 					(reference "#PWR013")
@@
 			)
 		)
-		(property "Value" "USB_C_Receptacle_USB2.0_16P"
+		(property "Value" "USB_C_16P"
 			(at 33.02 21.59 0)
 			(show_name no)
@@
 		)
 		(instances
-			(project "meshtastic-v0"
+			(project "meshthingy"
 				(path "/e4d6fcd6-7415-4955-88fd-f0e430797514/2c15135a-b809-49e8-b858-375c97ce8d4a"
 					(reference "J1")
@@
 		)
 		(instances
-			(project "meshtastic-v0"
+			(project "meshthingy"
 				(path "/e4d6fcd6-7415-4955-88fd-f0e430797514/2c15135a-b809-49e8-b858-375c97ce8d4a"
 					(reference "R2")
