File: Display.kicad_sch (KiCad schematic)
At the start: 3 parts, among them U1 DM-OLED096-636

Commit message: finalize
Parts:
- U1: value DM-OLED096-636 -> OLED096
Changed lines of the file:
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@@
 		)
 		(instances
-			(project "meshtastic-v0"
+			(project "meshthingy"
 				(path "/e4d6fcd6-7415-4955-88fd-f0e430797514/1f9f1566-46fa-44c7-a790-92c5c27114cc"
 					(reference "JP3")
@@
 		)
 		(instances
-			(project "meshtastic-v0"
+			(project "meshthingy"
 				(path "/e4d6fcd6-7415-4955-88fd-f0e430797514/1f9f1566-46fa-44c7-a790-92c5c27114cc"
 					(reference "#PWR045")
@@
 		)
 		(instances
-			(project "meshtastic-v0"
+			(project "meshthingy"
 				(path "/e4d6fcd6-7415-4955-88fd-f0e430797514/1f9f1566-46fa-44c7-a790-92c5c27114cc"
 					(reference "#PWR044")
@@
 			)
 		)
-		(property "Value" "DM-OLED096-636"
+		(property "Value" "OLED096"
 			(at 134.366 50.8 0)
 			(show_name no)
@@
 		)
 		(instances
-			(project "meshtastic-v0"
+			(project "meshthingy"
 				(path "/e4d6fcd6-7415-4955-88fd-f0e430797514/1f9f1566-46fa-44c7-a790-92c5c27114cc"
 					(reference "U1")
@@
 		)
 		(instances
-			(project "meshtastic-v0"
+			(project "meshthingy"
 				(path "/e4d6fcd6-7415-4955-88fd-f0e430797514/1f9f1566-46fa-44c7-a790-92c5c27114cc"
 					(reference "JP4")
