File: LORA.kicad_sch (KiCad schematic)
At the start: 4 parts, among them J4 Conn_Coaxial, U4 HT-RA62

Commit message: finalize
Parts:
- C10: value 100nF -> 100n; footprint Capacitor_SMD:C_0805_2012Metric_Pad1.18x1.45mm_HandSolder -> Capacitor_SMD:C_0805_2012Metric
- C9: value 10uF -> 10u; footprint Capacitor_SMD:C_0805_2012Metric_Pad1.18x1.45mm_HandSolder -> Capacitor_SMD:C_0805_2012Metric
- J4: value Conn_Coaxial -> SMA_Con
Connections:
- net SPI2_MISO: now also U4.13 (MISO); no longer U4.14 (MOSI)
- net SPI2_MOSI: now also U4.14 (MOSI); no longer U4.13 (MISO)
Changed lines of the file:
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@@
 	)
 	(hierarchical_label "LORA_RST"
-		(shape output)
+		(shape input)
 		(at 120.65 81.28 180)
 		(effects
@@
 	)
 	(hierarchical_label "SPI2_CLK"
-		(shape output)
+		(shape input)
 		(at 120.65 73.66 180)
 		(effects
@@
 	)
 	(hierarchical_label "SPI2_MOSI"
+		(shape input)
+		(at 120.65 68.58 180)
+		(effects
+			(font
+				(size 1.27 1.27)
+			)
+			(justify right)
+		)
+	)
+	(hierarchical_label "LORA_INT"
+		(shape output)
+		(at 146.05 71.12 0)
+		(effects
+			(font
+				(size 1.27 1.27)
+			)
+			(justify left)
+		)
+	)
+	(hierarchical_label "SPI2_MISO"
 		(shape output)
 		(at 120.65 71.12 180)
@@
 		)
 	)
-	(hierarchical_label "LORA_INT"
+	(hierarchical_label "SPI2_CS_N"
 		(shape input)
-		(at 146.05 71.12 0)
-		(effects
-			(font
-				(size 1.27 1.27)
-			)
-			(justify left)
-		)
-	)
-	(hierarchical_label "SPI2_MISO"
-		(shape input)
-		(at 120.65 68.58 180)
-		(effects
-			(font
-				(size 1.27 1.27)
-			)
-			(justify right)
-		)
-	)
-	(hierarchical_label "SPI2_CS_N"
-		(shape output)
 		(at 120.65 76.2 180)
 		(effects
@@
 	)
 	(hierarchical_label "LORA_BUSY"
-		(shape input)
+		(shape output)
 		(at 146.05 78.74 0)
 		(effects
@@
 		)
 		(instances
-			(project "meshtastic-v0"
+			(project "meshthingy"
 				(path "/e4d6fcd6-7415-4955-88fd-f0e430797514/1da3b465-1dc6-40ce-817b-2e6fcc10ae59"
 					(reference "#PWR06")
@@
 		)
 		(instances
-			(project "meshtastic-v0"
+			(project "meshthingy"
 				(path "/e4d6fcd6-7415-4955-88fd-f0e430797514/1da3b465-1dc6-40ce-817b-2e6fcc10ae59"
 					(reference "#PWR051")
@@
 			)
 		)
-		(property "Value" "10uF"
+		(property "Value" "10u"
 			(at 97.79 60.9599 0)
 			(show_name no)
@@
 			)
 		)
-		(property "Footprint" "Capacitor_SMD:C_0805_2012Metric_Pad1.18x1.45mm_HandSolder"
+		(property "Footprint" "Capacitor_SMD:C_0805_2012Metric"
 			(at 94.9452 63.5 0)
 			(hide yes)
@@
 		)
 		(instances
-			(project "meshtastic-v0"
+			(project "meshthingy"
 				(path "/e4d6fcd6-7415-4955-88fd-f0e430797514/1da3b465-1dc6-40ce-817b-2e6fcc10ae59"
 					(reference "C9")
@@
 		)
 		(instances
-			(project "meshtastic-v0"
+			(project "meshthingy"
 				(path "/e4d6fcd6-7415-4955-88fd-f0e430797514/1da3b465-1dc6-40ce-817b-2e6fcc10ae59"
 					(reference "#PWR031")
@@
 		)
 		(instances
-			(project "meshtastic-v0"
+			(project "meshthingy"
 				(path "/e4d6fcd6-7415-4955-88fd-f0e430797514/1da3b465-1dc6-40ce-817b-2e6fcc10ae59"
 					(reference "U4")
@@
 			)
 		)
-		(property "Value" "100nF"
+		(property "Value" "100n"
 			(at 110.49 60.9599 0)
 			(show_name no)
@@
 			)
 		)
-		(property "Footprint" "Capacitor_SMD:C_0805_2012Metric_Pad1.18x1.45mm_HandSolder"
+		(property "Footprint" "Capacitor_SMD:C_0805_2012Metric"
 			(at 107.6452 63.5 0)
 			(hide yes)
@@
 		)
 		(instances
-			(project "meshtastic-v0"
+			(project "meshthingy"
 				(path "/e4d6fcd6-7415-4955-88fd-f0e430797514/1da3b465-1dc6-40ce-817b-2e6fcc10ae59"
 					(reference "C10")
@@
 			)
 		)
-		(property "Value" "Conn_Coaxial"
+		(property "Value" "SMA_Con"
 			(at 166.37 65.0631 0)
 			(show_name no)
@@
 		)
 		(instances
-			(project "meshtastic-v0"
+			(project "meshthingy"
 				(path "/e4d6fcd6-7415-4955-88fd-f0e430797514/1da3b465-1dc6-40ce-817b-2e6fcc10ae59"
 					(reference "J4")
@@
 		)
 		(instances
-			(project "meshtastic-v0"
+			(project "meshthingy"
 				(path "/e4d6fcd6-7415-4955-88fd-f0e430797514/1da3b465-1dc6-40ce-817b-2e6fcc10ae59"
 					(reference "#PWR04")
