File: Microcontroller.kicad_sch (KiCad schematic)
At the start: 10 parts, among them U7 ESP32-S3-WROOM-1

Commit message: finalize
Parts:
- C1: value 100nF -> 100n; footprint Capacitor_SMD:C_0805_2012Metric_Pad1.18x1.45mm_HandSolder -> Capacitor_SMD:C_0805_2012Metric
- C2: value 10uF -> 10u; footprint Capacitor_SMD:C_0805_2012Metric_Pad1.18x1.45mm_HandSolder -> Capacitor_SMD:C_0805_2012Metric
Connections:
- net SPI2_MISO: now also U7.38 (IO2); no longer U7.39 (IO1)
- net SPI2_MOSI: now also U7.39 (IO1); no longer U7.38 (IO2)
Changed lines of the file:
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@@
+		)
+	)
+	(hierarchical_label "SPI2_MISO"
+		(shape input)
+		(at 105.41 59.69 180)
+		(effects
+			(font
+				(size 1.27 1.27)
+			)
+			(justify right)
 		)
 	)
@@
 		)
 	)
+	(hierarchical_label "SPI2_MOSI"
+		(shape output)
+		(at 105.41 57.15 180)
+		(effects
+			(font
+				(size 1.27 1.27)
+			)
+			(justify right)
+		)
+	)
 	(hierarchical_label "UART1_RX"
 		(shape input)
@@
 		)
 	)
-	(hierarchical_label "SPI2_MOSI"
-		(shape output)
-		(at 105.41 59.69 180)
-		(effects
-			(font
-				(size 1.27 1.27)
-			)
-			(justify right)
-		)
-	)
 	(hierarchical_label "I2C_SDA"
 		(shape bidirectional)
@@
 			)
 			(justify left)
-		)
-	)
-	(hierarchical_label "SPI2_MISO"
-		(shape input)
-		(at 105.41 57.15 180)
-		(effects
-			(font
-				(size 1.27 1.27)
-			)
-			(justify right)
 		)
 	)
@@
 		)
 		(instances
-			(project "meshtastic-v0"
+			(project "meshthingy"
 				(path "/e4d6fcd6-7415-4955-88fd-f0e430797514/b95685e3-53f8-4d4b-b7ad-2a266b169b28"
 					(reference "#PWR020")
@@
 		)
 		(instances
-			(project "meshtastic-v0"
+			(project "meshthingy"
 				(path "/e4d6fcd6-7415-4955-88fd-f0e430797514/b95685e3-53f8-4d4b-b7ad-2a266b169b28"
 					(reference "#PWR048")
@@
 		)
 		(instances
-			(project "meshtastic-v0"
+			(project "meshthingy"
 				(path "/e4d6fcd6-7415-4955-88fd-f0e430797514/b95685e3-53f8-4d4b-b7ad-2a266b169b28"
 					(reference "R19")
@@
 			)
 		)
-		(property "Value" "100nF"
+		(property "Value" "100n"
 			(at 93.98 44.4499 0)
 			(show_name no)
@@
 			)
 		)
-		(property "Footprint" "Capacitor_SMD:C_0805_2012Metric_Pad1.18x1.45mm_HandSolder"
+		(property "Footprint" "Capacitor_SMD:C_0805_2012Metric"
 			(at 91.1352 46.99 0)
 			(hide yes)
@@
 		)
 		(instances
-			(project "meshtastic-v0"
+			(project "meshthingy"
 				(path "/e4d6fcd6-7415-4955-88fd-f0e430797514/b95685e3-53f8-4d4b-b7ad-2a266b169b28"
 					(reference "C1")
@@
 		)
 		(instances
-			(project "meshtastic-v0"
+			(project "meshthingy"
 				(path "/e4d6fcd6-7415-4955-88fd-f0e430797514/b95685e3-53f8-4d4b-b7ad-2a266b169b28"
 					(reference "#PWR026")
@@
 		)
 		(instances
-			(project "meshtastic-v0"
+			(project "meshthingy"
 				(path "/e4d6fcd6-7415-4955-88fd-f0e430797514/b95685e3-53f8-4d4b-b7ad-2a266b169b28"
 					(reference "U7")
@@
 		)
 		(instances
-			(project "meshtastic-v0"
+			(project "meshthingy"
 				(path "/e4d6fcd6-7415-4955-88fd-f0e430797514/b95685e3-53f8-4d4b-b7ad-2a266b169b28"
 					(reference "RST1")
@@
 		)
 		(instances
-			(project "meshtastic-v0"
+			(project "meshthingy"
 				(path "/e4d6fcd6-7415-4955-88fd-f0e430797514/b95685e3-53f8-4d4b-b7ad-2a266b169b28"
 					(reference "BOOT1")
@@
 		)
 		(instances
-			(project "meshtastic-v0"
+			(project "meshthingy"
 				(path "/e4d6fcd6-7415-4955-88fd-f0e430797514/b95685e3-53f8-4d4b-b7ad-2a266b169b28"
 					(reference "R20")
@@
 		)
 		(instances
-			(project "meshtastic-v0"
+			(project "meshthingy"
 				(path "/e4d6fcd6-7415-4955-88fd-f0e430797514/b95685e3-53f8-4d4b-b7ad-2a266b169b28"
 					(reference "C17")
@@
 			)
 		)
-		(property "Value" "10uF"
+		(property "Value" "10u"
 			(at 81.28 44.4499 0)
 			(show_name no)
@@
 			)
 		)
-		(property "Footprint" "Capacitor_SMD:C_0805_2012Metric_Pad1.18x1.45mm_HandSolder"
+		(property "Footprint" "Capacitor_SMD:C_0805_2012Metric"
 			(at 78.4352 46.99 0)
 			(hide yes)
@@
 		)
 		(instances
-			(project "meshtastic-v0"
+			(project "meshthingy"
 				(path "/e4d6fcd6-7415-4955-88fd-f0e430797514/b95685e3-53f8-4d4b-b7ad-2a266b169b28"
 					(reference "C2")
@@
 		)
 		(instances
-			(project "meshtastic-v0"
+			(project "meshthingy"
 				(path "/e4d6fcd6-7415-4955-88fd-f0e430797514/b95685e3-53f8-4d4b-b7ad-2a266b169b28"
 					(reference "#PWR030")
@@
 		)
 		(instances
-			(project "meshtastic-v0"
+			(project "meshthingy"
 				(path "/e4d6fcd6-7415-4955-88fd-f0e430797514/b95685e3-53f8-4d4b-b7ad-2a266b169b28"
 					(reference "#PWR02")
@@
 		)
 		(instances
-			(project "meshtastic-v0"
+			(project "meshthingy"
 				(path "/e4d6fcd6-7415-4955-88fd-f0e430797514/b95685e3-53f8-4d4b-b7ad-2a266b169b28"
 					(reference "R10")
@@
 		)
 		(instances
-			(project "meshtastic-v0"
+			(project "meshthingy"
 				(path "/e4d6fcd6-7415-4955-88fd-f0e430797514/b95685e3-53f8-4d4b-b7ad-2a266b169b28"
 					(reference "R12")
@@
 		)
 		(instances
-			(project "meshtastic-v0"
+			(project "meshthingy"
 				(path "/e4d6fcd6-7415-4955-88fd-f0e430797514/b95685e3-53f8-4d4b-b7ad-2a266b169b28"
 					(reference "#PWR08")
@@
 		)
 		(instances
-			(project "meshtastic-v0"
+			(project "meshthingy"
 				(path "/e4d6fcd6-7415-4955-88fd-f0e430797514/b95685e3-53f8-4d4b-b7ad-2a266b169b28"
 					(reference "#PWR033")
@@
 		)
 		(instances
-			(project "meshtastic-v0"
+			(project "meshthingy"
 				(path "/e4d6fcd6-7415-4955-88fd-f0e430797514/b95685e3-53f8-4d4b-b7ad-2a266b169b28"
 					(reference "#PWR046")
