File: Peripherals.kicad_sch (KiCad schematic)
At the start: 22 parts, among them Q1 SI2302, Q4 SI2302

Commit message: finalize
Parts:
- removed CSN1: CSN, TestPoint:TestPoint_Pad_1.0x1.0mm, symbol Connector:TestPoint
- JP1: value SolderJumper_2_Open -> Vib_Motor_Conn
- LS1: value SMT-0927-S-14-R -> Buzzer 8.5x8.5x3
Connections:
- net GND: now also D2.1 (K); no longer R22.1
- net STATUS_LED: now also R22.2; no longer D2.1 (K)
- net at D2.2 (A): now also R22.1; no longer R22.2
Other:
- moved on the sheet: D2
