File: Power Management.kicad_sch (KiCad schematic)
At the start: 32 parts, among them Q2 Q_PNP_BEC, Q3 Q_NPN_BEC, U3 TPS62046DGQR, U5 Lever Switch TMHU26, U6 BQ24072RGT

Commit message: finalize
Parts:
- removed C12: 22u, Capacitor_SMD:C_0805_2012Metric, symbol Device:C
- removed D4, D6, D7, D8: 1N5819WS, Diode_SMD:D_SOD-323, symbol Diode:1N5819WS
- added C25: 22u, Capacitor_Tantalum_SMD:CP_EIA-3528-15_AVX-H, symbol Device:C_Polarized
- added D3, D4, D6, D7: 1N4148WS, Diode_SMD:D_SOD-323, symbol Diode:1N4148WS
- L2: value 6.8u -> 6.8uH
- Q2: value Q_PNP_BEC -> MMBT3906
- Q3: value Q_NPN_BEC -> MMBT3904
- R14: value 100k -> 47k
- R6: value 10k -> 47k
- U5: value Lever Switch TMHU26 -> TMHU26
Connections:
- net GND: now also C25.2
- net PGOOD: now also D3.1 (K), D4.1 (K)
- net PUSH_DWN: now also D6.1 (K), D7.1 (K)
- net PUSH_DWN_MCU: now also D6.2 (A)
- net P_GOOD: now also D3.2 (A)
- net VSYS: now also C25.1
- net at Q3.3 (C), R14.1, R8.1: now also D4.2 (A), D7.2 (A)
