File: GPS.kicad_sch (KiCad schematic)
At the start: 10 parts, among them J3 Conn_Coaxial, U2 ATGM336H, U8 AT24C32A

Commit message: finalize
Parts:
- added C22: 100n, Capacitor_SMD:C_0805_2012Metric, symbol Device:C
- added R24: 1k, Resistor_SMD:R_0805_2012Metric, symbol Device:R
- C18: value 10uF -> 10u; footprint Capacitor_SMD:C_0805_2012Metric_Pad1.18x1.45mm_HandSolder -> Capacitor_SMD:C_0805_2012Metric
- C19: value 100nF -> 100n; footprint Capacitor_SMD:C_0805_2012Metric_Pad1.18x1.45mm_HandSolder -> Capacitor_SMD:C_0805_2012Metric
Connections:
- net +3V3: now also C22.1, R24.1; no longer D1.2 (A)
- net GND: now also C22.2
- new net: D1.2 (A), R24.2

Commit message: fab ready
Parts:
- L1: footprint Inductor_SMD:L_0603_1608Metric -> Inductor_SMD:L_0402_1005Metric
Changed lines of the file:
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@@
 			)
 		)
-		(property "Footprint" "Inductor_SMD:L_0603_1608Metric"
+		(property "Footprint" "Inductor_SMD:L_0402_1005Metric"
 			(at 46.99 39.37 0)
 			(hide yes)
