File: meshthingy.kicad_pcb (KiCad board)
At the start: 2 copper layers, 71 x 46 mm, 96 parts, among them J1 USB_C_16P, J2 BATT_Con, J3 Conn_Coaxial, J4 SMA_Con, Q1 SI2302, Q2 MMBT3906, Q3 MMBT3904, Q4 SI2302, U1 OLED096, U10 LIS3DSHTR, U2 ATGM336H, U3 TPS62046DGQR, U4 HT-RA62, U5 TMHU26, U6 BQ24072RGT, U7 ESP32-S3-WROOM-1, U8 AT24C32A, U9 BME280

Commit message: fab ready
Parts:
- G***: moved to F.Cu
- G***: moved to B.Cu
- L1: footprint Inductor_SMD:L_0603_1608Metric -> Inductor_SMD:L_0402_1005Metric
- moved G*** 48.8 mm to (141.8, 105.5), turned to 180 degrees
- moved G*** 48.6 mm to (93.5, 105.8), turned to 0 degrees
- moved L1 0.31 mm to (88.5, 73.9)
Routing:
- net Net-(U2-VCC_RF): track 3.10 -> 3.71 mm
Other:
- board text added: "meow :3"
